File: Boards/revA/project/schematic.brd (EAGLE design)
At the start: 35.5 x 25.1 mm, 4 parts

Commit message: normal Push.
Parts:
- removed U$4: PIC18F26K20-X/ML, PIC18F26k20:QFN28_6X6MC
- removed VBAT1: (no value), BaseApp:BATTERY_HOLDER
- added C1: 0.1uF, SparkFun-Capacitors:0402-CAP
- added C10, C11, C12, C13, C14, C15, C4, C5, C6, C7, C8, C9: 1uF, SparkFun-Capacitors:0402-CAP
- added C2, C3: 12.5pF, SparkFun-Capacitors:0402-CAP
- added J1: (no value), baseOauth:2X3
- added JP1: (no value), SparkFun-Connectors:1X03
- added KP: 4X1-MEMBRANE-KEYPAD, baseOauth:4X1-MEMBRANE-KEYPAD
- added LCD: JHD508-12864, baseOauth:FSTN
- added LED1, LED2: (no value), adafruit:CHIP-LED0805
- added MCU: ATMEGA328-MMH, baseOauth:QFN45P400X400X100-29N
- added R1, R4: 1k, SparkFun-Passives:0402-RES
- added R2, R3: 10k, SparkFun-Passives:0402-RES
- added SOURCE: CR2025-CUSTOM-BASEAPP, baseOauth:CR2025-CUSTOM-BASEAPP
- added U$10, U$5, U$6, U$8, U$9: FIDUCIAL, adafruit:FIDUCIAL_1MM
- U$1: value JHD508-12864 -> ABS05; device baseOauth:FSTN -> baseOauth:ABS05
- U$2: value 4X1-MEMBRANE-KEYPAD -> FIDUCIAL; device baseOauth:4X1-MEMBRANE-KEYPAD -> adafruit:FIDUCIAL_1MM
- moved U$2 41.0 mm to (1.83, -2.13), turned to 0 degrees
- moved U$1 9.60 mm to (23.9, 5.33), flipped to the bottom, turned to 270 degrees
Connections:
- new net A0: LCD.P$19, MCU.11
- new net BTN1: KP.P$2, MCU.9
- new net BTN2: KP.P$3, MCU.8
- new net BTN3: KP.P$4, MCU.7
- new net DATA_L1: LED1.C, MCU.20, R1.2
- new net DATA_L2: LED2.C, MCU.21, R4.2
- new net GND: C1.2, C10.1, C14.1, C15.1, C2.1, C3.1, C4.1, C5.1, C6.1, C7.1, C8.1, C9.1, J1.6, JP1.1, LCD.P$15, MCU.18, MCU.29, MCU.4, R1.1, R4.1, SOURCE.1
- new net MISO: J1.1, MCU.14
- new net MOSI: J1.4, LCD.P$17, MCU.13
- new net N$1: C11.2, LCD.P$10
- new net N$10: C9.2, LCD.P$3
- new net N$11: C12.2, LCD.P$12
- new net N$12: C12.1, C13.1, LCD.P$11
- new net N$18: LCD.P$8
- new net N$19: C11.1, LCD.P$9
- new net N$2: C2.2, MCU.5, U$1.2
- new net N$23: C13.2, LCD.P$13
- new net N$3: C4.2, LCD.P$14
- new net N$4: C5.2, LCD.P$7
- new net N$5: C3.2, MCU.6, U$1.1
- new net N$7: C6.2, LCD.P$6
- new net N$8: C7.2, LCD.P$5
- new net N$9: C8.2, LCD.P$4
- new net RES: C10.2, LCD.P$20, MCU.10, R3.1
- new net RESET: J1.5, MCU.25, R2.1
- new net RXD: JP1.2, MCU.26
- new net SCK: J1.3, LCD.P$18, MCU.15
- new net SS: LCD.P$21, MCU.12
- new net TXD: JP1.3, MCU.27
- new net VDD: C1.1, C14.2, C15.2, J1.2, KP.P$1, LCD.P$1, LCD.P$16, LED1.A, LED2.A, MCU.16, MCU.17, MCU.3, R2.2, R3.2, SOURCE.2
- new net VR: LCD.P$2
Other:
- board size 35.5 x 25.1 mm -> 35 x 25 mm

Commit message: normal Push.
Parts:
- J1: device baseOauth:2X3 -> baseOauth:2X3_SMD
- JP1: device SparkFun-Connectors:1X03 -> SparkFun-Connectors:1X03_SMD_RA_MALE
- moved J1 28.0 mm to (4.27, 14.2), flipped to the top, turned to 90 degrees
- moved KP 24.9 mm to (30.0, 6.00), flipped to the bottom, turned to 90 degrees
- moved R2 19.6 mm to (23.5, 19.7), flipped to the top, turned to 270 degrees
- moved C15 19.3 mm to (14.7, 10.1), flipped to the top, turned to 45 degrees
- moved C13 18.2 mm to (19.8, 19.7), flipped to the top, turned to 270 degrees
- moved C12 17.9 mm to (18.6, 19.7), flipped to the top, turned to 270 degrees
- moved C4 17.7 mm to (21.0, 19.7), flipped to the top, turned to 270 degrees
- moved C14 17.2 mm to (22.3, 19.7), flipped to the top
- moved C11 17.1 mm to (16.3, 18.7), flipped to the top, turned to 0 degrees
- moved C5 15.1 mm to (13.9, 19.8), flipped to the top
- moved C7 15.1 mm to (11.4, 19.8), flipped to the top, turned to 270 degrees
- moved C8 15.0 mm to (8.53, 19.8), flipped to the top
- moved C6 13.3 mm to (12.6, 19.8), flipped to the top
- moved U$2 12.9 mm to (14.3, -5.18)
- moved C9 12.8 mm to (9.91, 19.8), flipped to the top, turned to 270 degrees
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Connections:
- new net VDD_GPIO: C14.2, LCD.P$16, MCU.28
- net VDD: no longer C14.2, LCD.P$16
Routing:
- net VDD: track 0.00 -> 111.8 mm, vias 0 -> 5
- net GND: track 0.00 -> 107.4 mm, vias 0 -> 9
- net RES: track 0.00 -> 45.4 mm
- net RESET: track 0.00 -> 43.0 mm, vias 0 -> 2
- net MOSI: track 0.00 -> 33.7 mm, vias 0 -> 3
- net SCK: track 0.00 -> 30.9 mm, vias 0 -> 3
- net DATA_L1: track 0.00 -> 26.4 mm, vias 0 -> 2
- net DATA_L2: track 0.00 -> 25.3 mm, vias 0 -> 1
- net VDD_GPIO: track 0.00 -> 17.4 mm, vias 0 -> 2
- net TXD: track 0.00 -> 16.2 mm
- net RXD: track 0.00 -> 14.9 mm
- net BTN1: track 0.00 -> 14.5 mm, vias 0 -> 1
- net SS: track 0.00 -> 13.0 mm, vias 0 -> 2
- net BTN2: track 0.00 -> 12.8 mm, vias 0 -> 1
- net MISO: track 0.00 -> 12.7 mm, vias 0 -> 2
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- added copper zone on layer 1, net GND
- added copper zone on layer 16, net GND

Commit message: normal Push.
Parts:
- removed J1: (no value), baseOauth:2X3_SMD
- removed JP1: (no value), SparkFun-Connectors:1X03_SMD_RA_MALE
- removed U$10, U$2, U$5, U$6, U$8, U$9: FIDUCIAL, adafruit:FIDUCIAL_1MM
- added SJ1: (no value), jumper:SJ_2
- added X1: 1365-12, con-leotronics:1365-12
- moved R3 12.8 mm to (3.96, 12.6), turned to 0 degrees
- moved LED1 8.06 mm to (29.0, 16.0)
- moved SOURCE 7.76 mm to (10.0, 10.0)
- moved C10 7.34 mm to (4.42, 18.1), turned to 270 degrees
- moved LED2 7.00 mm to (1.00, 16.0)
- moved R1 6.38 mm to (27.4, 18.2)
- moved KP 5.39 mm to (25.0, 4.00)
- moved R4 4.93 mm to (2.85, 18.2), turned to 270 degrees
- moved C1 3.48 mm to (27.1, 7.06)
- moved C9 3.21 mm to (7.16, 18.1)
- moved C5 3.21 mm to (11.1, 18.1)
- moved C6 3.21 mm to (9.91, 18.1)
- moved C7 3.21 mm to (8.69, 18.1)
- moved C8 3.21 mm to (5.79, 18.1)
- moved C13 3.14 mm to (17.1, 18.1)
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Connections:
- removed net N$18: LCD.P$8
- removed net VR: LCD.P$2
- new net N$6: C1.1, SJ1.1, SOURCE.2
- new net VIN: SJ1.3, X1.2
- net GND: now also X1.11, X1.4; no longer J1.6, JP1.1
- net MISO: now also X1.3; no longer J1.1
- net MOSI: now also X1.5; no longer J1.4
- net RESET: now also X1.10, X1.9; no longer J1.5
- net RXD: now also X1.6; no longer JP1.2
- net SCK: now also X1.7; no longer J1.3
- net TXD: now also X1.8; no longer JP1.3
- net VDD: now also SJ1.2, X1.1; no longer C1.1, J1.2, SOURCE.2
Routing:
- net VIN: track 0.00 -> 33.2 mm, vias 0 -> 2
- net VDD_GPIO: track 17.4 -> 34.9 mm
- net VDD: track 111.8 -> 99.1 mm, vias 5 -> 4
- net MISO: track 12.7 -> 25.1 mm
- net RES: track 45.4 -> 35.8 mm, vias 0 -> 2
- net N$6: track 0.00 -> 9.33 mm, vias 0 -> 1
- net MOSI: track 33.7 -> 25.4 mm
- net RESET: track 43.0 -> 48.5 mm, vias 2 -> 3
- net DATA_L2: track 25.3 -> 20.7 mm, vias 1 -> 3
- net SCK: track 30.9 -> 34.8 mm, vias 3 -> 4
- net GND: track 107.4 -> 104.0 mm, vias 9 -> 3
- net BTN1: track 14.5 -> 11.4 mm
- net RXD: track 14.9 -> 12.1 mm, vias 0 -> 2
- net SS: track 13.0 -> 10.3 mm
- net TXD: track 16.2 -> 13.5 mm, vias 0 -> 2
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- removed copper zone on layer 1, net GND
- removed copper zone on layer 16, net GND
Other:
- board size 35 x 25 mm -> 30 x 20 mm

Commit message: Normal Push.
Parts:
- removed SJ1: (no value), jumper:SJ_2
- removed U$1: ABS05, baseOauth:ABS05
- removed X1: 1365-12, con-leotronics:1365-12
- added ABS: ABS05, baseOauth:ABS05
- added EXTH: 1365-12, con-leotronics:1365-12
- moved R4 27.0 mm to (28.1, 8.74)
- moved C10 24.2 mm to (26.7, 8.74)
- moved C1 11.3 mm to (16.8, 2.47), turned to 225 degrees
- moved R2 9.54 mm to (28.1, 12.1), turned to 90 degrees
- moved C14 5.64 mm to (25.1, 18.2)
- moved C4 4.57 mm to (22.9, 18.2)
- moved C13 3.51 mm to (20.6, 18.2)
- moved C5 2.74 mm to (13.9, 18.2)
- moved C11 2.67 mm to (16.1, 18.2), turned to 270 degrees
- moved C12 2.44 mm to (18.3, 18.2)
- moved LED1 2.00 mm to (29.0, 18.0), turned to 0 degrees
- moved LED2 2.00 mm to (1.00, 18.0)
- moved C6 1.83 mm to (11.7, 18.2)
- moved C7 0.76 mm to (9.45, 18.2)
- moved C8 0.31 mm to (5.49, 18.2)
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- renumbered MCU to MCU-328
Connections:
- removed net N$6: C1.1, SJ1.1, SOURCE.2
- removed net VIN: SJ1.3, X1.2
- net GND: now also EXTH.11, EXTH.2, EXTH.4; no longer X1.11, X1.4
- net MISO: now also EXTH.3; no longer X1.3
- net MOSI: now also EXTH.5; no longer X1.5
- net N$2: now also ABS.2; no longer U$1.2
- net N$5: now also ABS.1; no longer U$1.1
- net RESET: now also EXTH.10, EXTH.9; no longer X1.10, X1.9
- net RXD: now also EXTH.6; no longer X1.6
- net SCK: now also EXTH.7; no longer X1.7
- net TXD: now also EXTH.8; no longer X1.8
- net VDD: now also C1.1, EXTH.1, SOURCE.2; no longer SJ1.2, X1.1
Routing:
- net GND: track 104.0 -> 0.00 mm, vias 3 -> 0
- net VDD: track 99.1 -> 0.00 mm, vias 4 -> 0
- net RESET: track 48.5 -> 0.00 mm, vias 3 -> 0
- net RES: track 35.8 -> 0.00 mm, vias 2 -> 0
- net VDD_GPIO: track 34.9 -> 0.00 mm, vias 2 -> 0
- net SCK: track 34.8 -> 0.00 mm, vias 4 -> 0
- net VIN: track 33.2 -> 0.00 mm, vias 2 -> 0
- net DATA_L1: track 26.7 -> 0.00 mm, vias 2 -> 0
- net MOSI: track 25.4 -> 0.00 mm, vias 3 -> 0
- net MISO: track 25.1 -> 0.00 mm, vias 2 -> 0
- net DATA_L2: track 20.7 -> 0.00 mm, vias 3 -> 0
- net TXD: track 13.5 -> 0.00 mm, vias 2 -> 0
- net BTN2: track 12.1 -> 0.00 mm, vias 1 -> 0
- net RXD: track 12.1 -> 0.00 mm, vias 2 -> 0
- net BTN1: track 11.4 -> 0.00 mm, vias 1 -> 0
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Other:
- board text added: "VDD"
