File: Boards/revA/project/schematic.brd (EAGLE design)
At the start: 30 x 20 mm, 27 parts

Commit message: Normal Push.
Parts:
- moved R4 27.5 mm to (2.24, 18.0)
- moved R3 22.3 mm to (25.6, 8.69), turned to 270 degrees
- moved R2 20.0 mm to (10.4, 2.90), turned to 225 degrees
- moved C9 3.35 mm to (3.81, 18.2)
- moved C7 1.83 mm to (7.62, 18.2)
- moved C6 1.83 mm to (9.91, 18.2)
- moved C5 1.68 mm to (12.2, 18.2)
- moved C11 0.72 mm to (15.3, 18.2), turned to 0 degrees
- moved C15 0.48 mm to (12.2, 10.6)
- moved C4 0.46 mm to (22.4, 18.2), turned to 90 degrees
- moved C12 0.46 mm to (17.8, 18.2)
- moved C13 0.46 mm to (20.1, 18.2)
- moved C14 0.46 mm to (24.7, 18.2)
- moved C8 0.46 mm to (5.94, 18.2)
- moved R1 0.46 mm to (27.0, 18.2)
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Connections:
- new net COG_RST: MCU-328.2, R3.2
- new net IRS: LCD.P$1, MCU-328.1
- net VDD: no longer LCD.P$1, R3.2
Routing:
- net VDD: track 0.00 -> 110.4 mm, vias 0 -> 4
- net GND: track 0.00 -> 83.8 mm, vias 0 -> 23
- net VDD_GPIO: track 0.00 -> 54.8 mm, vias 0 -> 4
- net DATA_L1: track 0.00 -> 44.1 mm, vias 0 -> 2
- net SCK: track 0.00 -> 30.7 mm, vias 0 -> 2
- net IRS: track 0.00 -> 29.5 mm, vias 0 -> 2
- net DATA_L2: track 0.00 -> 25.2 mm, vias 0 -> 2
- net MOSI: track 0.00 -> 23.6 mm, vias 0 -> 3
- net RESET: track 0.00 -> 19.5 mm, vias 0 -> 2
- net COG_RST: track 0.00 -> 18.3 mm, vias 0 -> 2
- net MISO: track 0.00 -> 16.9 mm, vias 0 -> 2
- net RES: track 0.00 -> 16.6 mm
- net N$3: track 0.00 -> 15.5 mm, vias 0 -> 2
- net N$9: track 0.00 -> 14.8 mm, vias 0 -> 2
- net TXD: track 0.00 -> 14.0 mm
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- added copper zone on layer 1, net GND
- added copper zone on layer 16, net GND
Other:
- board text added: "2014"
- board text added: "BASEOAUTH"
- board text added: "GND"
- board text added: "MISO"
- board text added: "MOSI"
- board text added: "NC"
- board text added: "RESET"
- board text added: "REV A"
- board text added: "RXD"
- board text added: "SCK"
- board text added: "TOP"
- board text added: "TXD"
