File: Boards/revA/project/schematic.sch (EAGLE design)
At the start: 34 parts

Commit message: normal Push.
Parts:
- J1: device baseOauth:M03X22X3_SILK_SM -> baseOauth:M03X2
- JP1: device SparkFun-Connectors:M03PTH -> SparkFun-Connectors:M03SMD_RA_MALE
Connections:
- new net VDD_GPIO: C14.2, LCD.VDD, MCU.PD2
- net VDD: no longer C14.2, LCD.VDD

Commit message: normal Push.
Parts:
- removed J1: (no value), baseOauth:M03X2
- removed JP1: (no value), SparkFun-Connectors:M03SMD_RA_MALE
- removed U$10, U$2, U$5, U$6, U$8, U$9: FIDUCIAL, adafruit:FIDUCIAL
- added SJ1: (no value), jumper:SJ2W
- added X1: 1365-12, con-leotronics:1365-12
Connections:
- removed net N$18: LCD.CAP4N
- removed net VR: LCD.VR
- new net N$6: C1.1, SJ1.1, SOURCE.VDD
- new net VIN: SJ1.3, X1-2.S
- net GND: now also X1-11.S, X1-4.S; no longer J1.6, JP1.1
- net MISO: now also X1-3.S; no longer J1.1
- net MOSI: now also X1-5.S; no longer J1.4
- net RESET: now also X1-10.S, X1-9.S; no longer J1.5
- net RXD: now also X1-6.S; no longer JP1.2
- net SCK: now also X1-7.S; no longer J1.3
- net TXD: now also X1-8.S; no longer JP1.3
- net VDD: now also SJ1.2, X1-1.S; no longer C1.1, J1.2, SOURCE.VDD

Commit message: Normal Push.
Parts:
- removed SJ1: (no value), jumper:SJ2W
- renumbered MCU to MCU-328, U$1 to ABS, X1 to EXTH
Connections:
- removed net N$6: C1.1, SJ1.1, SOURCE.VDD
- removed net VIN: EXTH-2.S, SJ1.3
- net GND: now also EXTH-2.S
- net VDD: now also C1.1, SOURCE.VDD; no longer SJ1.2

Commit message: Normal Push.
Connections:
- new net COG_RST: MCU-328.PD4, R3.2
- new net IRS: LCD.IRS, MCU-328.PD3
- net VDD: no longer LCD.IRS, R3.2
Changed lines of the file:
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@@
-</segment>
-<segment>
-<pinref part="LCD" gate="G$1" pin="IRS"/>
-<junction x="314.96" y="194.31"/>
-<wire x1="314.96" y1="194.31" x2="314.96" y2="189.23" width="0.1524" layer="91"/>
-<wire x1="314.96" y1="189.23" x2="317.5" y2="186.69" width="0.1524" layer="91"/>
-<wire x1="317.5" y1="186.69" x2="317.5" y2="182.88" width="0.1524" layer="91"/>
-<label x="317.5" y="182.88" size="1.016" layer="95" rot="R270" xref="yes"/>
-</segment>
-<segment>
-<pinref part="R3" gate="G$1" pin="2"/>
-<junction x="347.98" y="138.43"/>
-<wire x1="347.98" y1="138.43" x2="347.98" y2="132.08" width="0.1524" layer="91"/>
-<label x="347.98" y="132.08" size="1.016" layer="95" rot="R180" xref="yes"/>
 </segment>
 <segment>
@@
 </segment>
 </net>
+<net name="IRS" class="0">
+<segment>
+<pinref part="LCD" gate="G$1" pin="IRS"/>
+<junction x="314.96" y="194.31"/>
+<wire x1="314.96" y1="194.31" x2="314.96" y2="189.23" width="0.1524" layer="91"/>
+<wire x1="314.96" y1="189.23" x2="317.5" y2="186.69" width="0.1524" layer="91"/>
+<wire x1="317.5" y1="186.69" x2="317.5" y2="182.88" width="0.1524" layer="91"/>
+<label x="317.5" y="182.88" size="1.016" layer="95" rot="R270" xref="yes"/>
+</segment>
+<segment>
+<pinref part="MCU-328" gate="A" pin="PD3"/>
+<junction x="154.94" y="69.85"/>
+<wire x1="154.94" y1="69.85" x2="158.75" y2="69.85" width="0.1524" layer="91"/>
+<label x="158.75" y="69.85" size="1.016" layer="95" xref="yes"/>
+</segment>
+</net>
+<net name="COG_RST" class="0">
+<segment>
+<pinref part="R3" gate="G$1" pin="2"/>
+<junction x="347.98" y="138.43"/>
+<wire x1="347.98" y1="138.43" x2="341.63" y2="138.43" width="0.1524" layer="91"/>
+<label x="341.63" y="138.43" size="1.016" layer="95" rot="R180" xref="yes"/>
+</segment>
+<segment>
+<pinref part="MCU-328" gate="A" pin="PD4"/>
+<junction x="154.94" y="67.31"/>
+<wire x1="154.94" y1="67.31" x2="158.75" y2="67.31" width="0.1524" layer="91"/>
+<label x="158.75" y="67.31" size="1.016" layer="95" xref="yes"/>
+</segment>
+</net>
