File: Boards/revB/schematic.sch (EAGLE design)
At the start: 29 parts, among them X1 1365-12

Commit message: normal Push.
Parts:
- removed 16MHZ: ABS05, baseOauth:ABS05
- removed SJ1: (no value), jumper:SJ2W
- removed X1: 1365-12, con-leotronics:1365-12
- added 32MHZ: ABS05, baseOauth:ABS05
- added ANT: ANTENNA2SMD3, SparkFun-RF:ANTENNA2SMD3
- added C17, C18: 12pF, SparkFun-Capacitors:CAP0402-CAP
- added C19: 2.2nF, SparkFun-Capacitors:CAP0402-CAP
- added C23: 47nF, SparkFun-Capacitors:CAP0402-CAP
- added C24: 1uF, SparkFun-Capacitors:CAP0402-CAP
- added C25: 4.7uF, SparkFun-Capacitors:CAP0402-CAP
- added KHZ: CRYSTAL, abracon:CRYSTAL
- added L4: 10uH,50mA, SparkFun-Passives:INDUCTOR0402
- added L5: 15nH,50mA, SparkFun-Passives:INDUCTOR0402
- added LED3: (no value), led:LEDSML0603
- added R5: 220, SparkFun-Passives:RESISTOR0402-RES
- added TP1, TP2, TP3, TP4: TPTP06SQ, testpad:TPTP06SQ
- added U$1: 2450BM14E0003_BALUN, baseOauth:2450BM14E0003_BALUN
- R2: value 10k -> 12k
Connections:
- removed net N$6: C1.1, SJ1.1, SOURCE.VDD
- removed net RESET: R2.1, X1-10.S, X1-9.S
- removed net RXD: X1-6.S
- removed net TXD: X1-8.S
- removed net VDD_GPIO: C14.2, LCD.VDD
- removed net VIN: SJ1.3, X1-2.S
- new net ANT1: NRF.ANT1, U$1.3
- new net ANT2: NRF.ANT2, U$1.4
- new net FEED: ANT.SIGNAL, U$1.1
- new net N$16: C23.1, NRF.DEC2
- new net N$17: C17.2, KHZ.1, NRF.P0.27
- new net N$18: L4.2, NRF.DCC
- new net N$2: C18.2, KHZ.2, NRF.P0.26
- new net N$20: L4.1, L5.2
- new net N$21: LED3.C, R5.2
- new net SWDCLK: NRF.SWDCLK, R2.1, TP4.TP
- new net SWDIO/NRESET: NRF.SWDIO/NRESET, TP3.TP
- new net TORCHLED: NRF.P0.18, R5.1
- new net VDD_COG: C14.2, LCD.IRS, LCD.VDD, NRF.P0.20, R3.2
- new net VDD_PA: C19.1, NRF.VDD_PA, U$1.5
- new net VDD_PT: LED1.A, LED2.A, NRF.P0.19
- net A0: now also NRF.P0.09
- net AVDD: now also C24.1, L5.1
- net BTN1: now also NRF.P0.14
- net BTN2: now also NRF.P0.15
- net BTN3: now also NRF.P0.16
- net DATA_L1: now also NRF.P0.02
- net DATA_L2: now also NRF.P0.01
- net GND: now also C17.1, C18.1, C19.2, C23.2, C24.2, C25.2, NRF.VSS, R2.2, TP1.TP, U$1.2, U$1.6; no longer X1-11.S, X1-4.S
- net MISO: now also NRF.P0.12; no longer X1-3.S
- net MOSI: now also NRF.P0.11; no longer X1-5.S
- net N$13: now also 32MHZ.1; no longer 16MHZ.1
- net N$14: now also 32MHZ.2; no longer 16MHZ.2
- net RES: now also NRF.P0.08
- net SCK: now also NRF.P0.13; no longer X1-7.S
- net SS: now also NRF.P0.10
- net VDD: now also C1.1, C25.1, LED3.A, NRF.VDD, SOURCE.VDD, TP2.TP; no longer LCD.IRS, LED1.A, LED2.A, R2.2, R3.2, SJ1.2, X1-1.S
Other:
- note added: "1"
- note added: "2.4-2.485 GHz chip Antenna"
- note added: "B"
- note added: "BaseApp"
- note added: "Headers"
- note added: "SoC NRF81522"
- note removed: "Microcontroller"
- moved on the sheet: C1, C10, C11, C12, C13, C14, C15, C16, C2, C3, C4, C5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

Commit message: Normal Push.
Parts:
- renumbered LED3 to TRCH, U$1 to BU
Connections:
- new net COG_IRS: LCD.IRS, NRF.P0.17
- new net COG_RST: NRF.P0.21, R3.2
- net GND: now also NRF.DIE_PAD
- net VDD_COG: no longer LCD.IRS, R3.2
Changed lines of the file:
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@@
 <setting verticaltext="up"/>
 </settings>
-<grid distance="0.1" unitdist="inch" unit="inch" style="lines" multiple="1" display="no" altdistance="0.01" altunitdist="inch" altunit="inch"/>
+<grid distance="0.05" unitdist="inch" unit="inch" style="lines" multiple="1" display="yes" altdistance="0.01" altunitdist="inch" altunit="inch"/>
 <layers>
 <layer number="1" name="Top" color="4" fill="1" visible="no" active="no"/>
@@
 <part name="TP3" library="testpad" deviceset="TP" device="TP06SQ"/>
 <part name="TP4" library="testpad" deviceset="TP" device="TP06SQ"/>
-<part name="LED3" library="led" deviceset="LED" device="SML0603"/>
+<part name="TRCH" library="led" deviceset="LED" device="SML0603"/>
 <part name="R5" library="SparkFun-Passives" deviceset="RESISTOR" device="0402-RES" value="220"/>
 <part name="ANT" library="SparkFun-RF" deviceset="ANTENNA2" device="SMD3" value="ANTENNA2SMD3"/>
-<part name="U$1" library="baseOauth" deviceset="2450BM14E0003_BALUN" device=""/>
+<part name="BU" library="baseOauth" deviceset="2450BM14E0003_BALUN" device=""/>
 <part name="C19" library="SparkFun-Capacitors" deviceset="CAP" device="0402-CAP" value="2.2nF"/>
 </parts>
@@
 <text x="124.46" y="186.69" size="3.81" layer="94">Keypad</text>
 <text x="222.25" y="109.22" size="3.81" layer="94">COG LCD</text>
-<text x="24.13" y="175.26" size="3.81" layer="94">Photo Transistor</text>
+<text x="16.51" y="173.99" size="3.81" layer="94">Photo Transistor</text>
 <text x="269.24" y="7.62" size="2.54" layer="94">B</text>
 <text x="256.54" y="7.62" size="2.54" layer="94">1</text>
@@
 <instance part="TP3" gate="G$1" x="160.02" y="142.24" rot="R90"/>
 <instance part="TP4" gate="G$1" x="160.02" y="147.32" rot="R90"/>
-<instance part="LED3" gate="G$1" x="105.41" y="139.7" rot="R90"/>
+<instance part="TRCH" gate="G$1" x="105.41" y="139.7" rot="R90"/>
 <instance part="R5" gate="G$1" x="118.11" y="139.7" rot="R180"/>
 <instance part="ANT" gate="G$1" x="54.61" y="148.59"/>
-<instance part="U$1" gate="G$1" x="33.02" y="144.78" rot="R180"/>
+<instance part="BU" gate="G$1" x="33.02" y="144.78" rot="R180"/>
 <instance part="C19" gate="G$1" x="15.24" y="132.08"/>
 </instances>
@@
 </segment>
 <segment>
-<pinref part="U$1" gate="G$1" pin="6"/>
+<pinref part="BU" gate="G$1" pin="6"/>
 <junction x="25.4" y="139.7"/>
 <wire x1="25.4" y1="139.7" x2="21.59" y2="139.7" width="0.1524" layer="91"/>
@@
 </segment>
 <segment>
-<pinref part="U$1" gate="G$1" pin="2"/>
+<pinref part="BU" gate="G$1" pin="2"/>
 <junction x="40.64" y="144.78"/>
 <wire x1="40.64" y1="144.78" x2="44.45" y2="144.78" width="0.1524" layer="91"/>
@@
 <wire x1="15.24" y1="129.54" x2="15.24" y2="125.73" width="0.1524" layer="91"/>
 <label x="15.24" y="125.73" size="0.8128" layer="95" xref="yes"/>
+</segment>
+<segment>
+<pinref part="NRF" gate="G$1" pin="DIE_PAD"/>
+<junction x="92.71" y="46.99"/>
+<wire x1="92.71" y1="46.99" x2="92.71" y2="49.53" width="0.1524" layer="91"/>
+<wire x1="92.71" y1="49.53" x2="95.25" y2="49.53" width="0.1524" layer="91"/>
+<label x="95.25" y="49.53" size="1.016" layer="95" xref="yes"/>
 </segment>
 </net>
@@
 </segment>
 <segment>
-<pinref part="LED3" gate="G$1" pin="A"/>
+<pinref part="TRCH" gate="G$1" pin="A"/>
 <junction x="102.87" y="139.7"/>
 <wire x1="102.87" y1="139.7" x2="100.33" y2="139.7" width="0.1524" layer="91"/>
@@
 </segment>
 <segment>
-<pinref part="R3" gate="G$1" pin="2"/>
-<junction x="237.49" y="124.46"/>
-<wire x1="237.49" y1="124.46" x2="234.95" y2="124.46" width="0.1524" layer="91"/>
-<label x="234.95" y="124.46" size="1.016" layer="95" rot="R180" xref="yes"/>
-</segment>
-<segment>
-<pinref part="LCD" gate="G$1" pin="IRS"/>
-<junction x="217.17" y="168.91"/>
-<wire x1="217.17" y1="168.91" x2="217.17" y2="163.83" width="0.1524" layer="91"/>
-<wire x1="217.17" y1="163.83" x2="219.71" y2="161.29" width="0.1524" layer="91"/>
-<wire x1="219.71" y1="161.29" x2="219.71" y2="157.48" width="0.1524" layer="91"/>
-<label x="219.71" y="157.48" size="1.016" layer="95" rot="R270" xref="yes"/>
-</segment>
-<segment>
 <pinref part="NRF" gate="G$1" pin="P0.20"/>
 <junction x="130.81" y="46.99"/>
@@
 </segment>
 <segment>
-<pinref part="U$1" gate="G$1" pin="4"/>
+<pinref part="BU" gate="G$1" pin="4"/>
 <junction x="25.4" y="149.86"/>
 <wire x1="25.4" y1="149.86" x2="21.59" y2="149.86" width="0.1524" layer="91"/>
@@
 </segment>
 <segment>
-<pinref part="U$1" gate="G$1" pin="3"/>
+<pinref part="BU" gate="G$1" pin="3"/>
 <junction x="40.64" y="149.86"/>
 <wire x1="40.64" y1="149.86" x2="44.45" y2="149.86" width="0.1524" layer="91"/>
@@
 <segment>
 <label x="44.45" y="139.7" size="0.8128" layer="95" xref="yes"/>
-<pinref part="U$1" gate="G$1" pin="1"/>
+<pinref part="BU" gate="G$1" pin="1"/>
 <junction x="40.64" y="139.7"/>
 <wire x1="44.45" y1="139.7" x2="40.64" y2="139.7" width="0.1524" layer="91"/>
@@
 </segment>
 <segment>
-<pinref part="U$1" gate="G$1" pin="5"/>
+<pinref part="BU" gate="G$1" pin="5"/>
 <junction x="25.4" y="144.78"/>
 <label x="15.24" y="144.78" size="0.8128" layer="95" rot="R180" xref="yes"/>
@@
 <net name="N$21" class="0">
 <segment>
-<pinref part="LED3" gate="G$1" pin="C"/>
+<pinref part="TRCH" gate="G$1" pin="C"/>
 <junction x="110.49" y="139.7"/>
 <pinref part="R5" gate="G$1" pin="2"/>
@@
 </segment>
 </net>
+<net name="COG_IRS" class="0">
+<segment>
+<pinref part="NRF" gate="G$1" pin="P0.17"/>
+<junction x="130.81" y="39.37"/>
+<wire x1="130.81" y1="39.37" x2="137.16" y2="39.37" width="0.1524" layer="91"/>
+<wire x1="137.16" y1="39.37" x2="137.16" y2="38.1" width="0.1524" layer="91"/>
+<label x="137.16" y="38.1" size="0.8128" layer="95" rot="R270" xref="yes"/>
+</segment>
+<segment>
+<pinref part="LCD" gate="G$1" pin="IRS"/>
+<junction x="217.17" y="168.91"/>
+<wire x1="217.17" y1="168.91" x2="217.17" y2="163.83" width="0.1524" layer="91"/>
+<wire x1="217.17" y1="163.83" x2="219.71" y2="161.29" width="0.1524" layer="91"/>
+<wire x1="219.71" y1="161.29" x2="219.71" y2="157.48" width="0.1524" layer="91"/>
+<label x="219.71" y="157.48" size="1.016" layer="95" rot="R270" xref="yes"/>
+</segment>
+</net>
+<net name="COG_RST" class="0">
+<segment>
+<pinref part="R3" gate="G$1" pin="2"/>
+<junction x="237.49" y="124.46"/>
+<wire x1="237.49" y1="124.46" x2="234.95" y2="124.46" width="0.1524" layer="91"/>
+<label x="234.95" y="124.46" size="1.016" layer="95" rot="R180" xref="yes"/>
+</segment>
+<segment>
+<pinref part="NRF" gate="G$1" pin="P0.21"/>
+<junction x="107.95" y="82.55"/>
+<wire x1="107.95" y1="82.55" x2="107.95" y2="86.36" width="0.1524" layer="91"/>
+<label x="107.95" y="86.36" size="1.016" layer="95" rot="R90" xref="yes"/>
+</segment>
+</net>
