File: Boards/revB/schematic.brd (EAGLE design)
At the start: 30 x 20 mm, 29 parts, among them X1 1365-12

Commit message: normal Push.
Parts:
- removed 16MHZ: ABS05, baseOauth:ABS05
- removed SJ1: (no value), jumper:SJ_2
- removed X1: 1365-12, con-leotronics:1365-12
- added 32MHZ: ABS05, baseOauth:ABS05
- added ANT: ANTENNA2SMD3, SparkFun-RF:ANTENNA-CHIP4
- added C17, C18: 12pF, SparkFun-Capacitors:0402-CAP
- added C19: 2.2nF, SparkFun-Capacitors:0402-CAP
- added C23: 47nF, SparkFun-Capacitors:0402-CAP
- added C24: 1uF, SparkFun-Capacitors:0402-CAP
- added C25: 4.7uF, SparkFun-Capacitors:0402-CAP
- added KHZ: CRYSTAL, abracon:ABS05
- added L4: 10uH,50mA, SparkFun-Passives:C0402
- added L5: 15nH,50mA, SparkFun-Passives:C0402
- added LED3: (no value), led:SML0603
- added R5: 220, SparkFun-Passives:0402-RES
- added TP1, TP2, TP3, TP4: TPTP06SQ, testpad:TP06SQ
- added U$1: 2450BM14E0003_BALUN, baseOauth:6PCPADS
- R2: value 10k -> 12k
- moved R2 23.4 mm to (0.76, 5.94)
- moved C16 13.0 mm to (9.60, 4.72), turned to 90 degrees
- moved C3 9.11 mm to (13.4, 7.21), turned to 180 degrees
- moved NRF 8.89 mm to (5.87, 8.91), turned to 270 degrees
- moved C2 6.46 mm to (13.4, 5.93), turned to 180 degrees
- moved C1 3.66 mm to (23.5, 7.21)
- moved KP 3.30 mm to (27.7, 5.83)
- moved R3 2.33 mm to (4.42, 14.9), turned to 270 degrees
- moved C15 2.11 mm to (13.4, 8.43), turned to 0 degrees
- moved LED1 1.78 mm to (29.0, 17.8)
- moved LED2 1.78 mm to (1.00, 17.8)
- moved C8 1.68 mm to (7.47, 18.1)
- moved C9 1.22 mm to (5.94, 18.1)
- moved C11 0.46 mm to (13.6, 17.7)
Connections:
- removed net N$6: C1.1, SJ1.1, SOURCE.2
- removed net RESET: R2.1, X1.10, X1.9
- removed net RXD: X1.6
- removed net TXD: X1.8
- removed net VDD_GPIO: C14.2, LCD.P$16
- removed net VIN: SJ1.3, X1.2
- new net ANT1: NRF.31, U$1.P$3
- new net ANT2: NRF.32, U$1.P$4
- new net FEED: ANT.SIG, U$1.P$1
- new net N$16: C23.1, NRF.29
- new net N$17: C17.2, KHZ.P$1, NRF.46
- new net N$18: L4.2, NRF.2
- new net N$2: C18.2, KHZ.P$2, NRF.45
- new net N$20: L4.1, L5.2
- new net N$21: LED3.C, R5.2
- new net SWDCLK: NRF.24, R2.1, TP4.TP
- new net SWDIO/NRESET: NRF.23, TP3.TP
- new net TORCHLED: NRF.26, R5.1
- new net VDD_COG: C14.2, LCD.P$1, LCD.P$16, NRF.28, R3.2
- new net VDD_PA: C19.1, NRF.30, U$1.P$5
- new net VDD_PT: LED1.A, LED2.A, NRF.27
- net A0: now also NRF.15
- net AVDD: now also C24.1, L5.1
- net BTN1: now also NRF.20
- net BTN2: now also NRF.21
- net BTN3: now also NRF.22
- net DATA_L1: now also NRF.6
- net DATA_L2: now also NRF.5
- net GND: now also C17.1, C18.1, C19.2, C23.2, C24.2, C25.2, NRF.13, R2.2, TP1.TP, U$1.P$2, U$1.P$6; no longer X1.11, X1.4
- net MISO: now also NRF.18; no longer X1.3
- net MOSI: now also NRF.17; no longer X1.5
- net N$13: now also 32MHZ.1; no longer 16MHZ.1
- net N$14: now also 32MHZ.2; no longer 16MHZ.2
- net RES: now also NRF.14
- net SCK: now also NRF.19; no longer X1.7
- net SS: now also NRF.16
- net VDD: now also C1.1, C25.1, LED3.A, NRF.1, SOURCE.2, TP2.TP; no longer LCD.P$1, LED1.A, LED2.A, R2.2, R3.2, SJ1.2, X1.1

Commit message: LED ADDED and Component Placed.
Parts:
- moved LED3 46.3 mm to (28.2, 1.22), turned to 0 degrees
- moved R5 45.2 mm to (25.1, 1.22), turned to 0 degrees
- moved C17 2.59 mm to (16.0, 11.1)
- moved C18 2.59 mm to (16.0, 9.75)
- moved C15 2.59 mm to (16.0, 8.43)
- moved C2 2.59 mm to (16.0, 5.93)
- moved C3 2.59 mm to (16.0, 7.21)
- moved C14 0.76 mm to (20.3, 18.1)
- moved C4 0.61 mm to (18.9, 18.1)
- moved C13 0.46 mm to (17.5, 18.1)
- moved C8 0.46 mm to (7.01, 18.1)
- moved C7 0.30 mm to (8.38, 18.1)
- moved C9 0.30 mm to (5.64, 18.1)
- moved L4 0.30 mm to (9.14, 15.2)
- moved C12 0.30 mm to (16.2, 18.1)
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
Commit message: Normal Push.
Parts:
- removed LED3: (no value), led:SML0603
- removed U$1: 2450BM14E0003_BALUN, baseOauth:6PCPADS
- added BU: 2450BM14E0003_BALUN, baseOauth:6PCPADS
- added TRCH: (no value), led:SML0603
- moved C10 21.1 mm to (23.5, 9.45), turned to 0 degrees
- moved R3 20.5 mm to (23.6, 7.77), turned to 180 degrees
- moved C24 15.0 mm to (1.07, 14.3), turned to 270 degrees
- moved L5 9.19 mm to (3.51, 14.3), turned to 0 degrees
- moved TP2 8.10 mm to (8.38, 13.0)
- moved ANT 6.66 mm to (11.8, 1.37), turned to 0 degrees
- moved 32MHZ 6.07 mm to (16.9, 5.11)
- moved KHZ 5.79 mm to (16.9, 10.4)
- moved C14 5.64 mm to (25.9, 18.0)
- moved C4 4.73 mm to (23.6, 18.0)
- moved C1 3.81 mm to (23.5, 11.0)
- moved C13 3.81 mm to (21.3, 18.1)
- moved C2 3.68 mm to (19.4, 4.40)
- moved TP1 3.68 mm to (2.13, 13.1)
- moved C11 3.42 mm to (16.8, 18.9)
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Connections:
- new net COG_IRS: LCD.P$1, NRF.25
- new net COG_RST: NRF.40, R3.2
- net ANT1: now also BU.P$3; no longer U$1.P$3
- net ANT2: now also BU.P$4; no longer U$1.P$4
- net FEED: now also BU.P$1; no longer U$1.P$1
- net GND: now also BU.P$2, BU.P$6, NRF.GND; no longer U$1.P$2, U$1.P$6
- net N$21: now also TRCH.C; no longer LED3.C
- net VDD: now also TRCH.A; no longer LED3.A
- net VDD_COG: no longer LCD.P$1, R3.2
- net VDD_PA: now also BU.P$5; no longer U$1.P$5
Other:
- board text added: "MHz"
- board text added: "kHz"

Commit message: Normal Push.
Parts:
- moved C25 11.6 mm to (19.7, 19.2)
- moved C11 9.55 mm to (19.5, 28.0)
- moved C13 9.55 mm to (24.1, 27.3)
- moved C4 9.55 mm to (26.4, 27.1)
- moved C5 9.55 mm to (16.3, 27.1)
- moved C6 9.55 mm to (14.0, 27.1)
- moved C7 9.55 mm to (11.7, 27.1)
- moved C8 9.55 mm to (9.45, 27.1)
- moved C9 9.55 mm to (7.16, 27.3)
- moved LED1 9.55 mm to (31.7, 26.9)
- moved LED2 9.55 mm to (3.74, 26.9)
- moved R1 9.55 mm to (31.0, 27.2)
- moved R4 9.55 mm to (4.98, 27.2)
- moved C12 9.55 mm to (21.8, 27.3)
- moved C14 9.55 mm to (28.7, 27.1)
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Routing:
- net GND: track 0.00 -> 145.7 mm, vias 0 -> 5
- net SS: track 0.00 -> 47.0 mm, vias 0 -> 3
- net RES: track 0.00 -> 47.0 mm, vias 0 -> 3
- net VDD: track 0.00 -> 46.6 mm, vias 0 -> 2
- net VDD_COG: track 0.00 -> 41.7 mm, vias 0 -> 5
- net VDD_PT: track 0.00 -> 40.5 mm, vias 0 -> 2
- net BTN2: track 0.00 -> 35.2 mm, vias 0 -> 1
- net SCK: track 0.00 -> 34.1 mm, vias 0 -> 1
- net DATA_L1: track 0.00 -> 33.5 mm, vias 0 -> 1
- net COG_IRS: track 0.00 -> 32.8 mm, vias 0 -> 1
- net AVDD: track 0.00 -> 32.6 mm, vias 0 -> 2
- net TORCHLED: track 0.00 -> 23.9 mm, vias 0 -> 2
- net COG_RST: track 0.00 -> 20.3 mm, vias 0 -> 2
- net N$17: track 0.00 -> 14.7 mm, vias 0 -> 2
- net N$14: track 0.00 -> 14.5 mm, vias 0 -> 2
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Other:
- board size 30 x 20 mm -> 35 x 30 mm

Commit message: Normal Push.rev B Routed
Parts:
- moved TP4 1.89 mm to (5.64, 8.99)
- moved BU 1.38 mm to (11.4, 4.27), turned to 90 degrees
- moved C19 0.61 mm to (7.32, 4.88)
- moved TP3 0.61 mm to (5.64, 10.1)
- moved C3 0.48 mm to (26.1, 11.0)
- moved C18 0.22 mm to (26.1, 14.9)
- moved C5 0.15 mm to (16.3, 27.3)
- moved C6 0.15 mm to (14.0, 27.3)
- moved C7 0.15 mm to (11.7, 27.3)
- moved C8 0.15 mm to (9.45, 27.3)
Routing:
- net VDD: track 46.6 -> 107.7 mm, vias 2 -> 4
- net BTN3: track 0.00 -> 42.3 mm, vias 0 -> 1
- net A0: track 0.00 -> 31.7 mm, vias 0 -> 3
- net BTN1: track 0.00 -> 30.1 mm, vias 0 -> 1
- net MOSI: track 0.00 -> 25.4 mm, vias 0 -> 1
- net VDD_PT: track 40.5 -> 64.9 mm, vias 2 -> 3
- net AVDD: track 32.6 -> 51.8 mm, vias 2 -> 4
- net DATA_L2: track 3.82 -> 22.2 mm, vias 1 -> 2
- net TORCHLED: track 23.9 -> 40.4 mm
- net GND: track 145.7 -> 160.4 mm, vias 5 -> 30
- net N$5: track 0.00 -> 11.9 mm
- net VDD_COG: track 41.7 -> 52.4 mm
- net N$16: track 0.00 -> 9.38 mm
- net RES: track 47.0 -> 56.0 mm, vias 3 -> 2
- net SS: track 47.0 -> 38.9 mm
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- added copper zone on layer 1, net GND
- added copper zone on layer 16, net GND
